Commit message: panda movit added

File: panda_description/urdf/panda.gazebo.xacro (robot description, xacro)
@@ -10,5 +10,5 @@
     <!-- Link0 -->
     <gazebo reference="${robot_name}_link0">
-      <material>Gazebo/Grey</material>
+      <material>Gazebo/White</material>
       <mu1>0.2</mu1>
       <mu2>0.2</mu2>
@@ -16,5 +16,5 @@
     <!-- Link1 -->
     <gazebo reference="${robot_name}_link1">
-      <material>Gazebo/Orange</material>
+      <material>Gazebo/White</material>
       <mu1>0.2</mu1>
       <mu2>0.2</mu2>
@@ -22,5 +22,5 @@
     <!-- Link2 -->
     <gazebo reference="${robot_name}_link2">
-      <material>Gazebo/Orange</material>
+      <material>Gazebo/White</material>
       <mu1>0.2</mu1>
       <mu2>0.2</mu2>
@@ -28,5 +28,5 @@
     <!-- Link3 -->
     <gazebo reference="${robot_name}_link3">
-      <material>Gazebo/Orange</material>
+      <material>Gazebo/White</material>
       <mu1>0.2</mu1>
       <mu2>0.2</mu2>
@@ -34,5 +34,5 @@
     <!-- Link4 -->
     <gazebo reference="${robot_name}_link4">
-      <material>Gazebo/Orange</material>
+      <material>Gazebo/White</material>
       <mu1>0.2</mu1>
       <mu2>0.2</mu2>
@@ -40,5 +40,5 @@
     <!-- Link5 -->
     <gazebo reference="${robot_name}_link5">
-      <material>Gazebo/Orange</material>
+      <material>Gazebo/White</material>
       <mu1>0.2</mu1>
       <mu2>0.2</mu2>
@@ -46,5 +46,5 @@
     <!-- Link6 -->
     <gazebo reference="${robot_name}_link6">
-      <material>Gazebo/Orange</material>
+      <material>Gazebo/White</material>
       <mu1>0.2</mu1>
       <mu2>0.2</mu2>
